File: Hardware/Actuator/NomadBLDC/PCB_V1.2/kicad/PCB_V1.2/PCB_V1.2.sch (KiCad schematic (older format))
At the start: 66 parts, among them Q1 TPH, Q2 TPH, Q3 TPH, Q4 TPH, Q5 TPH, Q6 TPH

Commit message: Changes to schematic
Parts:
- C1, C2, C3, C4, C5, C6, C7, C8: value 10 -> 10uF, 50v
- C10, C13: value .1 uF -> 0.1uF, 50v
- C12: value 22 uF -> 22uF
- C14: value 47 nF -> 47nF, 50v
- C15: value 1 uF -> 1uF
- C16: value 1 uF -> 1uF, 50v
- C17: value 4.7 -> 4.7uF
- C26, C27, C28: value .1 uF -> .1uF
- C9: value 10 uF, 50v -> 10uF, 50v
Other:
- note added: "All caps 10v except unless specifically labeled 50v"
- note added: "CAN\n"
- note added: "MOSFETS\n"
- note added: "Programing\n"
- moved on the sheet: C1, C10, C11, C12, C13, C14, C15, C16, C17, C18, C19, C2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
