File: Hardware/Actuator/NomadBLDC/PCBV1.3_CSD/KICAD/PCB_V1.3_CSD 2/PCB_V1.3_CSD.kicad_pcb (KiCad board)
At the start: 4 copper layers, 42.7 x 37.2 mm, 66 parts, among them J1 Conn_01x03, J2 USB_B_Micro, U1 CSD88599Q5DC, U3 CSD88599Q5DC, U4 CSD88599Q5DC

Commit message: updated some files
Parts:
- C15, C2, C4, C5, C6: value 0.1uF -> 100nF
- R10, R8: value 22 -> 200
- moved CAN1 0.11 mm to (86.5, 72.2)
Connections:
- AS5047P1 pad 10: Net-(AS5047P1-Pad10) -> (no net)
- AS5047P1 pad 14: Net-(AS5047P1-Pad14) -> (no net)
- AS5047P1 pad 5: Net-(AS5047P1-Pad5) -> (no net)
- AS5047P1 pad 6: Net-(AS5047P1-Pad6) -> (no net)
- AS5047P1 pad 7: Net-(AS5047P1-Pad7) -> (no net)
- AS5047P1 pad 8: Net-(AS5047P1-Pad8) -> (no net)
- AS5047P1 pad 9: Net-(AS5047P1-Pad9) -> (no net)
- DRV1 pad 28: /FAULT -> (no net)
- DRV1 pad 34: /CAL -> (no net)
- DRV1 pad 46: Net-(DRV1-Pad46) -> (no net)
- DRV1 pad 48: Net-(DRV1-Pad48) -> (no net)
- LDFM1 pad 2: Net-(LDFM1-Pad2) -> (no net)
- LDFM1 pad 3: Net-(LDFM1-Pad3) -> (no net)
- R7 pad 2: Net-(R7-Pad2) -> (no net)
- R9 pad 1: Net-(R9-Pad1) -> (no net)
- STM1 pad 11: Net-(STM1-Pad11) -> (no net)
- STM1 pad 2: Net-(STM1-Pad2) -> (no net)
- STM1 pad 24: Net-(STM1-Pad24) -> (no net)
- STM1 pad 26: Net-(STM1-Pad26) -> (no net)
- STM1 pad 27: Net-(STM1-Pad27) -> (no net)
- STM1 pad 28: Net-(STM1-Pad28) -> (no net)
- STM1 pad 29: Net-(STM1-Pad29) -> (no net)
- STM1 pad 3: Net-(STM1-Pad3) -> (no net)
- STM1 pad 33: Net-(STM1-Pad33) -> (no net)
- STM1 pad 34: Net-(STM1-Pad34) -> (no net)
- STM1 pad 35: Net-(STM1-Pad35) -> (no net)
- STM1 pad 36: Net-(STM1-Pad36) -> (no net)
- STM1 pad 37: Net-(STM1-Pad37) -> (no net)
- STM1 pad 38: Net-(STM1-Pad38) -> (no net)
- STM1 pad 39: Net-(STM1-Pad39) -> (no net)
- STM1 pad 4: Net-(STM1-Pad4) -> (no net)
- STM1 pad 54: Net-(STM1-Pad54) -> (no net)
- STM1 pad 55: Net-(STM1-Pad55) -> (no net)
- STM1 pad 56: Net-(STM1-Pad56) -> (no net)
- STM1 pad 57: Net-(STM1-Pad57) -> (no net)
- STM1 pad 58: Net-(STM1-Pad58) -> (no net)
- STM1 pad 59: Net-(STM1-Pad59) -> (no net)
Other:
- board text added: "CAN"
- board text added: "V1.2: QJ/OW"
- board text added: "V1.3: QJ/OW"
- board text removed: "V1.3_CSD: QJ/OW"
