File: Hardware/Actuator/NomadBLDC/PCBV1.3_CSD/KICAD/PCB_V1.3_CSD 2/PCB_V1.3_CSD.sch (KiCad schematic (older format))
At the start: 66 parts, among them J1 Conn_01x03, J2 USB_B_Micro, U1 CSD88599Q5DC, U3 CSD88599Q5DC, U4 CSD88599Q5DC

Commit message: updated some files
Parts:
- AS5047P1: MANUFACTURER ams -> (none); MPN AS5147P-HTSM -> (none); POPULATE 0 -> (none)
- C1: MANUFACTURER Murata Electronics -> (none); MPN GRM155R60J475ME87D -> (none); POPULATE 1 -> (none)
- C10: MANUFACTURER Yageo -> (none); MPN CC0402JRX7R9BB473 -> (none); POPULATE 1 -> (none)
- C11, C12: MANUFACTURER Yageo -> (none); MPN CC0603JRX7R9BB104 -> (none); POPULATE 1 -> (none)
- C13, C3: MANUFACTURER KEMET -> (none); MPN C0402C105K8PACTU -> (none); POPULATE 1 -> (none)
- C14: symbol PCB_V1.2-rescue:C-USC0402K-HKCV4-eagle-import -> PCB_V1.2-rescue:C-USC0402-HKCV4-eagle-import; MANUFACTURER KEMET -> (none); MPN C0402C105K8PACTU -> (none); POPULATE 1 -> (none)
- C15, C4, C5, C6: value 0.1uF -> 100nF; MANUFACTURER KEMET -> (none); MPN C0402C104K8PAC7411 -> (none); POPULATE 1 -> (none)
- C17, C19, C7: MANUFACTURER Murata Electronics -> (none); MPN GRM188R61A226ME15J -> (none); POPULATE 1 -> (none)
- C18: MANUFACTURER TDK -> (none); MPN CGA3E3X5R1H105K080AB -> (none); POPULATE 1 -> (none)
- C2: value 0.1uF -> 100nF; symbol PCB_V1.2-rescue:C-USC0402K-HKCV4-eagle-import -> PCB_V1.2-rescue:C-USC0402-HKCV4-eagle-import; MANUFACTURER KEMET -> (none); MPN C0402C104K8PAC7411 -> (none); POPULATE 1 -> (none)
- C22, C8, C9: MANUFACTURER KEMET -> (none); MPN C0402C104K8PAC7411 -> (none); POPULATE 1 -> (none)
- C23, C24, C25, C26, C27, C28, C29, C30, C31, C32, C33, C34, C35, C36, C37: MANUFACTURER Murata Electronics -> (none); MPN GRT31CR61H106ME01L -> (none); POPULATE 1 -> (none)
- CAN1: MANUFACTURER Microchip Technology -> (none); MPN MCP2542FDT-H/MNY -> (none); POPULATE 1 -> (none)
- CHOKE1: MANUFACTURER Pulse Electronics -> (none); MPN PE-0603FB601ST -> (none); POPULATE 1 -> (none)
- D1: MANUFACTURER Diodes Incorporated -> (none); MPN MBR0580S1-7 -> (none); POPULATE 1 -> (none)
- DRV1: MANUFACTURER Texas Instruments -> (none); MPN DRV8323RSRGZT -> (none); POPULATE 1 -> (none)
- J1: MANUFACTURER JST Sales America Inc. -> (none); MPN BM03B-SURS-TF(LF)(SN) -> (none); POPULATE 1 -> (none)
- J2: MANUFACTURER GCT -> (none); MPN USB3076-30-A -> (none); POPULATE 1 -> (none)
- JP1: POPULATE 0 -> (none)
- L1: MANUFACTURER Taiyo Yuden -> (none); MPN NRH3012T220MNV -> (none); POPULATE 1 -> (none)
- LDFM1: symbol PCB_V1.3_CSD-rescue:LDFM-Regulator_Linear -> Regulator_Linear:LDFM; MANUFACTURER STMicroelectronics -> (none); MPN LDFM33PUR -> (none); POPULATE 1 -> (none)
- LED1, LED2: MANUFACTURER Lite-On -> (none); MPN LTST-C191KRKT -> (none); POPULATE 1 -> (none)
- PROG1: MANUFACTURER JST Sales America Inc. -> (none); MPN SM08B-SRSS-TB(LF)(SN) -> (none); POPULATE 1 -> (none)
- R1: MANUFACTURER Yageo -> (none); MPN RC0402DR-07150KL -> (none); POPULATE 1 -> (none)
- R10, R8: value 22 -> 200; MANUFACTURER Yageo -> (none); MPN RC0402JR-0722RL -> (none); POPULATE 1 -> (none)
- R12, R13, R14: MANUFACTURER ROHM Semiconductor -> (none); MPN PMR25HZPFV1L00 -> (none); POPULATE 1 -> (none)
- R2, R3, TERM1: MANUFACTURER Yageo -> (none); MPN RC0402JR-07200RL -> (none); POPULATE 1 -> (none)
- R4, R6, R7, R9: MANUFACTURER Yageo -> (none); MPN RT0402DRE0710KL -> (none); POPULATE 1 -> (none)
- R5: MANUFACTURER Yageo -> (none); MPN RC0402FR-0754K9L -> (none); POPULATE 1 -> (none)
- STM1: MANUFACTURER STMicroelectronics -> (none); MPN STM32F446RET6 -> (none); POPULATE 1 -> (none)
- U1, U3, U4: symbol PCB_V1.3_CSD-rescue:CSD88599Q5DC-CSD88599Q5DC -> CSD88599Q5DC:CSD88599Q5DC; Field4 (none) -> Unavailable; Field5 (none) -> None; Field6 (none) -> Texas Instruments; Field7 (none) -> VSON-22 Texas Instruments; Field8 (none) -> CSD88599Q5DC; MANUFACTURER Texas Instruments -> (none); MPN CSD88599Q5DC -> (none); POPULATE 1 -> (none)
- XTAL1: MANUFACTURER Murata Electronics -> (none); MPN CSTNE8M00GH5L000R0 -> (none); POPULATE 1 -> (none)
