Commit message: Working on sim.

File: Software/Simulation/Gazebo/models/Nomad/Nomad.urdf (robot description, URDF)
Before this commit: robot Nomad, 25 links, 24 joints
Links:
- removed link b_foot_FL__1
- removed link b_foot_FR__1
- removed link b_foot_RL__1
- removed link b_foot_RR__1
- removed link b_haa_motor_FL__1
- removed link b_haa_motor_FR__1
- removed link b_haa_motor_RL__1
- removed link b_haa_motor_RR__1
- removed link b_hfe_motor_FL__1
- removed link b_hfe_motor_FR__1
- removed link b_hfe_motor_RL__1
- removed link b_hfe_motor_RR__1
- removed link b_kfe_motor_FL__1
- removed link b_kfe_motor_FR__1
- removed link b_kfe_motor_RL__1
- removed link b_kfe_motor_RR__1
- removed link b_lower_leg_FL__1
- removed link b_lower_leg_FR__1
- removed link b_lower_leg_RL__1
- removed link b_lower_leg_RR__1
- removed link b_upper_leg_FL__1
- removed link b_upper_leg_FR__1
- removed link b_upper_leg_RL__1
- removed link b_upper_leg_RR__1
- added link b_foot_FL, mass 0.07686399002843429; collision mesh filename=package://Nomad/meshes/b_foot_FL.stl scale=0.001 0.001 0.001; visual mesh filename=package://Nomad/meshes/b_foot_FL.stl scale=0.001 0.001 0.001
- added link b_foot_FR, mass 0.07686399002843429; collision mesh filename=package://Nomad/meshes/b_foot_FR.stl scale=0.001 0.001 0.001; visual mesh filename=package://Nomad/meshes/b_foot_FR.stl scale=0.001 0.001 0.001
- added link b_foot_RL, mass 0.07686399002843429; collision mesh filename=package://Nomad/meshes/b_foot_RL.stl scale=0.001 0.001 0.001; visual mesh filename=package://Nomad/meshes/b_foot_RL.stl scale=0.001 0.001 0.001
- added link b_foot_RR, mass 0.07686399002843429; collision mesh filename=package://Nomad/meshes/b_foot_RR.stl scale=0.001 0.001 0.001; visual mesh filename=package://Nomad/meshes/b_foot_RR.stl scale=0.001 0.001 0.001
- added link b_haa_motor_FL, mass 0.22819661408568134; collision mesh filename=package://Nomad/meshes/b_haa_motor_FL.stl scale=0.001 0.001 0.001; visual mesh filename=package://Nomad/meshes/b_haa_motor_FL.stl scale=0.001 0.001 0.001
- added link b_haa_motor_FR, mass 0.22819661408568134; collision mesh filename=package://Nomad/meshes/b_haa_motor_FR.stl scale=0.001 0.001 0.001; visual mesh filename=package://Nomad/meshes/b_haa_motor_FR.stl scale=0.001 0.001 0.001
- added link b_haa_motor_RL, mass 0.22819661408568134; collision mesh filename=package://Nomad/meshes/b_haa_motor_RL.stl scale=0.001 0.001 0.001; visual mesh filename=package://Nomad/meshes/b_haa_motor_RL.stl scale=0.001 0.001 0.001
- added link b_haa_motor_RR, mass 0.22819661408568134; collision mesh filename=package://Nomad/meshes/b_haa_motor_RR.stl scale=0.001 0.001 0.001; visual mesh filename=package://Nomad/meshes/b_haa_motor_RR.stl scale=0.001 0.001 0.001
- added link b_hfe_motor_FL, mass 0.2875872093499024; collision mesh filename=package://Nomad/meshes/b_hfe_motor_FL.stl scale=0.001 0.001 0.001; visual mesh filename=package://Nomad/meshes/b_hfe_motor_FL.stl scale=0.001 0.001 0.001
- added link b_hfe_motor_FR, mass 0.2875872093499024; collision mesh filename=package://Nomad/meshes/b_hfe_motor_FR.stl scale=0.001 0.001 0.001; visual mesh filename=package://Nomad/meshes/b_hfe_motor_FR.stl scale=0.001 0.001 0.001
- added link b_hfe_motor_RL, mass 0.2875872093499024; collision mesh filename=package://Nomad/meshes/b_hfe_motor_RL.stl scale=0.001 0.001 0.001; visual mesh filename=package://Nomad/meshes/b_hfe_motor_RL.stl scale=0.001 0.001 0.001
- added link b_hfe_motor_RR, mass 0.2875872093499024; collision mesh filename=package://Nomad/meshes/b_hfe_motor_RR.stl scale=0.001 0.001 0.001; visual mesh filename=package://Nomad/meshes/b_hfe_motor_RR.stl scale=0.001 0.001 0.001
- added link b_kfe_motor_FL, mass 0.30243979231772933; collision mesh filename=package://Nomad/meshes/b_kfe_motor_FL.stl scale=0.001 0.001 0.001; visual mesh filename=package://Nomad/meshes/b_kfe_motor_FL.stl scale=0.001 0.001 0.001
- added link b_kfe_motor_FR, mass 0.30244037793017975; collision mesh filename=package://Nomad/meshes/b_kfe_motor_FR.stl scale=0.001 0.001 0.001; visual mesh filename=package://Nomad/meshes/b_kfe_motor_FR.stl scale=0.001 0.001 0.001
- added link b_kfe_motor_RL, mass 0.30243979231772933; collision mesh filename=package://Nomad/meshes/b_kfe_motor_RL.stl scale=0.001 0.001 0.001; visual mesh filename=package://Nomad/meshes/b_kfe_motor_RL.stl scale=0.001 0.001 0.001
- added link b_kfe_motor_RR, mass 0.30244037793017975; collision mesh filename=package://Nomad/meshes/b_kfe_motor_RR.stl scale=0.001 0.001 0.001; visual mesh filename=package://Nomad/meshes/b_kfe_motor_RR.stl scale=0.001 0.001 0.001
- added link b_lower_leg_FL, mass 0.10027511378483192; collision mesh filename=package://Nomad/meshes/b_lower_leg_FL.stl scale=0.001 0.001 0.001; visual mesh filename=package://Nomad/meshes/b_lower_leg_FL.stl scale=0.001 0.001 0.001
- added link b_lower_leg_FR, mass 0.10027511378483192; collision mesh filename=package://Nomad/meshes/b_lower_leg_FR.stl scale=0.001 0.001 0.001; visual mesh filename=package://Nomad/meshes/b_lower_leg_FR.stl scale=0.001 0.001 0.001
- added link b_lower_leg_RL, mass 0.10027511378483192; collision mesh filename=package://Nomad/meshes/b_lower_leg_RL.stl scale=0.001 0.001 0.001; visual mesh filename=package://Nomad/meshes/b_lower_leg_RL.stl scale=0.001 0.001 0.001
- added link b_lower_leg_RR, mass 0.10027511378483192; collision mesh filename=package://Nomad/meshes/b_lower_leg_RR.stl scale=0.001 0.001 0.001; visual mesh filename=package://Nomad/meshes/b_lower_leg_RR.stl scale=0.001 0.001 0.001
- added link b_upper_leg_FL, mass 0.28719650938086905; collision mesh filename=package://Nomad/meshes/b_upper_leg_FL.stl scale=0.001 0.001 0.001; visual mesh filename=package://Nomad/meshes/b_upper_leg_FL.stl scale=0.001 0.001 0.001
- added link b_upper_leg_FR, mass 0.28719862886504943; collision mesh filename=package://Nomad/meshes/b_upper_leg_FR.stl scale=0.001 0.001 0.001; visual mesh filename=package://Nomad/meshes/b_upper_leg_FR.stl scale=0.001 0.001 0.001
- added link b_upper_leg_RL, mass 0.28719650938086905; collision mesh filename=package://Nomad/meshes/b_upper_leg_RL.stl scale=0.001 0.001 0.001; visual mesh filename=package://Nomad/meshes/b_upper_leg_RL.stl scale=0.001 0.001 0.001
- added link b_upper_leg_RR, mass 0.28719862886504943; collision mesh filename=package://Nomad/meshes/b_upper_leg_RR.stl scale=0.001 0.001 0.001; visual mesh filename=package://Nomad/meshes/b_upper_leg_RR.stl scale=0.001 0.001 0.001
- link base_link: mass 2.199914 -> 2.199913990617033; geometry collision mesh filename=package://Nomad/meshes/base_link.stl scale=0.001 0.001 0.001; visual mesh filename=package://Nomad/meshes/base_link.stl scale=0.001 0.001 0.001
Joints:
- joint j_base_link_haa_FL: child b_haa_motor_FL__1 -> b_haa_motor_FL
- joint j_base_link_haa_FR: child b_haa_motor_FR__1 -> b_haa_motor_FR
- joint j_base_link_haa_RL: child b_haa_motor_RL__1 -> b_haa_motor_RL
- joint j_base_link_haa_RR: child b_haa_motor_RR__1 -> b_haa_motor_RR
- joint j_haa_FL: axis 0.01 0.0 0.0 -> -1.0 0.0 0.0; child b_hfe_motor_FL__1 -> b_hfe_motor_FL; parent b_haa_motor_FL__1 -> b_haa_motor_FL
- joint j_haa_FR: axis 0.01 0.0 -0.0 -> -1.0 0.0 -0.0; child b_hfe_motor_FR__1 -> b_hfe_motor_FR; parent b_haa_motor_FR__1 -> b_haa_motor_FR
- joint j_haa_RL: axis -0.01 -0.0 -0.0 -> 1.0 -0.0 -0.0; child b_hfe_motor_RL__1 -> b_hfe_motor_RL; parent b_haa_motor_RL__1 -> b_haa_motor_RL
- joint j_haa_RR: axis -0.01 -0.0 -0.0 -> 1.0 -0.0 -0.0; child b_hfe_motor_RR__1 -> b_hfe_motor_RR; parent b_haa_motor_RR__1 -> b_haa_motor_RR
- joint j_hfe_FL: axis -0.0 0.01 0.0 -> -0.0 -1.0 0.0; child b_kfe_motor_FL__1 -> b_kfe_motor_FL; parent b_hfe_motor_FL__1 -> b_hfe_motor_FL
- joint j_hfe_FR: axis 0.0 0.01 0.0 -> 0.0 1.0 0.0; child b_kfe_motor_FR__1 -> b_kfe_motor_FR; parent b_hfe_motor_FR__1 -> b_hfe_motor_FR
- joint j_hfe_RL: axis -0.0 -0.01 0.0 -> -0.0 -1.0 0.0; child b_kfe_motor_RL__1 -> b_kfe_motor_RL; parent b_hfe_motor_RL__1 -> b_hfe_motor_RL
- joint j_hfe_RR: axis 0.0 -0.01 -0.0 -> 0.0 1.0 -0.0; child b_kfe_motor_RR__1 -> b_kfe_motor_RR; parent b_hfe_motor_RR__1 -> b_hfe_motor_RR
- joint j_hfe_to_shoulder_FL: child b_upper_leg_FL__1 -> b_upper_leg_FL; parent b_kfe_motor_FL__1 -> b_kfe_motor_FL
- joint j_hfe_to_shoulder_FR: child b_upper_leg_FR__1 -> b_upper_leg_FR; parent b_kfe_motor_FR__1 -> b_kfe_motor_FR
- joint j_hfe_to_shoulder_RL: child b_upper_leg_RL__1 -> b_upper_leg_RL; parent b_kfe_motor_RL__1 -> b_kfe_motor_RL
- joint j_hfe_to_shoulder_RR: child b_upper_leg_RR__1 -> b_upper_leg_RR; parent b_kfe_motor_RR__1 -> b_kfe_motor_RR
- joint j_kfe_FL: axis 0.0 -0.01 0.0 -> 0.0 -1.0 0.0; child b_lower_leg_FL__1 -> b_lower_leg_FL; parent b_upper_leg_FL__1 -> b_upper_leg_FL
- joint j_kfe_FR: axis -0.0 -0.01 -0.0 -> -0.0 1.0 -0.0; child b_lower_leg_FR__1 -> b_lower_leg_FR; parent b_upper_leg_FR__1 -> b_upper_leg_FR
- joint j_kfe_RL: axis -0.0 -0.01 -0.0 -> -0.0 -1.0 -0.0; child b_lower_leg_RL__1 -> b_lower_leg_RL; parent b_upper_leg_RL__1 -> b_upper_leg_RL
- joint j_kfe_RR: axis 0.0 -0.01 0.0 -> 0.0 1.0 0.0; child b_lower_leg_RR__1 -> b_lower_leg_RR; parent b_upper_leg_RR__1 -> b_upper_leg_RR
- joint j_knee_to_foot_FL: child b_foot_FL__1 -> b_foot_FL; parent b_lower_leg_FL__1 -> b_lower_leg_FL
- joint j_knee_to_foot_FR: child b_foot_FR__1 -> b_foot_FR; parent b_lower_leg_FR__1 -> b_lower_leg_FR
- joint j_knee_to_foot_RL: child b_foot_RL__1 -> b_foot_RL; parent b_lower_leg_RL__1 -> b_lower_leg_RL
- joint j_knee_to_foot_RR: child b_foot_RR__1 -> b_foot_RR; parent b_lower_leg_RR__1 -> b_lower_leg_RR

Commit message: Collision URDF improvements

File: Software/Simulation/Gazebo/models/Nomad/Nomad.urdf (robot description, URDF)
Before this commit: robot Nomad, 25 links, 24 joints
Links:
- link b_foot_FL: geometry collision sphere radius=0.025; visual mesh filename=package://Nomad/meshes/b_foot_FL.stl scale=0.001 0.001 0.001
- link b_foot_FR: geometry collision sphere radius=0.025; visual mesh filename=package://Nomad/meshes/b_foot_FR.stl scale=0.001 0.001 0.001
- link b_foot_RL: geometry collision sphere radius=0.025; visual mesh filename=package://Nomad/meshes/b_foot_RL.stl scale=0.001 0.001 0.001
- link b_foot_RR: geometry collision sphere radius=0.025; visual mesh filename=package://Nomad/meshes/b_foot_RR.stl scale=0.001 0.001 0.001
- link b_haa_motor_FL: geometry visual mesh filename=package://Nomad/meshes/b_haa_motor_FL.stl scale=0.001 0.001 0.001
- link b_haa_motor_FR: geometry visual mesh filename=package://Nomad/meshes/b_haa_motor_FR.stl scale=0.001 0.001 0.001
- link b_haa_motor_RL: geometry visual mesh filename=package://Nomad/meshes/b_haa_motor_RL.stl scale=0.001 0.001 0.001
- link b_haa_motor_RR: geometry visual mesh filename=package://Nomad/meshes/b_haa_motor_RR.stl scale=0.001 0.001 0.001
- link b_hfe_motor_FL: geometry collision cylinder length=0.053 radius=0.05; visual mesh filename=package://Nomad/meshes/b_hfe_motor_FL.stl scale=0.001 0.001 0.001
- link b_hfe_motor_FR: geometry collision cylinder length=0.053 radius=0.05; visual mesh filename=package://Nomad/meshes/b_hfe_motor_FR.stl scale=0.001 0.001 0.001
- link b_hfe_motor_RL: geometry collision cylinder length=0.053 radius=0.05; visual mesh filename=package://Nomad/meshes/b_hfe_motor_RL.stl scale=0.001 0.001 0.001
- link b_hfe_motor_RR: geometry collision cylinder length=0.053 radius=0.05; visual mesh filename=package://Nomad/meshes/b_hfe_motor_RR.stl scale=0.001 0.001 0.001
- link b_kfe_motor_FL: geometry collision cylinder length=0.075 radius=0.05
- link b_kfe_motor_FR: geometry collision cylinder length=0.075 radius=0.05; visual mesh filename=package://Nomad/meshes/b_kfe_motor_FR.stl scale=0.001 0.001 0.001
- link b_kfe_motor_RL: geometry collision cylinder length=0.075 radius=0.05; visual mesh filename=package://Nomad/meshes/b_kfe_motor_RL.stl scale=0.001 0.001 0.001
- link b_kfe_motor_RR: geometry collision cylinder length=0.075 radius=0.05; visual mesh filename=package://Nomad/meshes/b_kfe_motor_RR.stl scale=0.001 0.001 0.001
- link b_lower_leg_FL: geometry visual mesh filename=package://Nomad/meshes/b_lower_leg_FL.stl scale=0.001 0.001 0.001
- link b_lower_leg_FR: geometry visual mesh filename=package://Nomad/meshes/b_lower_leg_FR.stl scale=0.001 0.001 0.001
- link b_lower_leg_RL: geometry visual mesh filename=package://Nomad/meshes/b_lower_leg_RL.stl scale=0.001 0.001 0.001
- link b_lower_leg_RR: geometry visual mesh filename=package://Nomad/meshes/b_lower_leg_RR.stl scale=0.001 0.001 0.001
- link b_upper_leg_FL: geometry collision cylinder length=1.075 radius=0.14; visual mesh filename=package://Nomad/meshes/b_upper_leg_FL.stl scale=0.001 0.001 0.001
- link b_upper_leg_FR: geometry visual mesh filename=package://Nomad/meshes/b_upper_leg_FR.stl scale=0.001 0.001 0.001
- link b_upper_leg_RL: geometry visual mesh filename=package://Nomad/meshes/b_upper_leg_RL.stl scale=0.001 0.001 0.001
- link b_upper_leg_RR: geometry visual mesh filename=package://Nomad/meshes/b_upper_leg_RR.stl scale=0.001 0.001 0.001
- link base_link: geometry collision box size=0.440 0.260 0.140

Commit message: More collsions

File: Software/Simulation/Gazebo/models/Nomad/Nomad.urdf (robot description, URDF)
Before this commit: robot Nomad, 25 links, 24 joints
Links:
- link b_lower_leg_FL: geometry collision cylinder length=0.250 radius=0.02; visual mesh filename=package://Nomad/meshes/b_lower_leg_FL.stl scale=0.001 0.001 0.001
- link b_upper_leg_FL: geometry collision box size=.05 .030 .25; visual mesh filename=package://Nomad/meshes/b_upper_leg_FL.stl scale=0.001 0.001 0.001

Commit message: Simplifed URDF collision model is complete (good enough)

File: Software/Simulation/Gazebo/models/Nomad/Nomad.urdf (robot description, URDF)
Before this commit: robot Nomad, 25 links, 24 joints
Links:
- link b_kfe_motor_FL: geometry collision cylinder length=0.075 radius=0.05; visual mesh filename=package://Nomad/meshes/b_kfe_motor_FL.stl scale=0.001 0.001 0.001
- link b_lower_leg_FL: geometry collision cylinder length=0.260 radius=0.01; visual mesh filename=package://Nomad/meshes/b_lower_leg_FL.stl scale=0.001 0.001 0.001
- link b_lower_leg_FR: geometry collision cylinder length=0.260 radius=0.01; visual mesh filename=package://Nomad/meshes/b_lower_leg_FR.stl scale=0.001 0.001 0.001
- link b_lower_leg_RL: geometry collision cylinder length=0.260 radius=0.01; visual mesh filename=package://Nomad/meshes/b_lower_leg_RL.stl scale=0.001 0.001 0.001
- link b_lower_leg_RR: geometry collision cylinder length=0.260 radius=0.01; visual mesh filename=package://Nomad/meshes/b_lower_leg_RR.stl scale=0.001 0.001 0.001
- link b_upper_leg_FR: geometry collision box size=.05 .030 .25; visual mesh filename=package://Nomad/meshes/b_upper_leg_FR.stl scale=0.001 0.001 0.001
- link b_upper_leg_RL: geometry collision box size=.05 .030 .25; visual mesh filename=package://Nomad/meshes/b_upper_leg_RL.stl scale=0.001 0.001 0.001
- link b_upper_leg_RR: geometry collision box size=.05 .030 .25; visual mesh filename=package://Nomad/meshes/b_upper_leg_RR.stl scale=0.001 0.001 0.001
- link base_link: geometry collision box size=0.440 0.260 0.140; visual mesh filename=package://Nomad/meshes/base_link.stl scale=0.001 0.001 0.001

Commit message: Simulation Interface is Connected to Simulation

File: Software/Simulation/Gazebo/models/Nomad/Nomad.urdf (robot description, URDF)
Before this commit: robot Nomad, 25 links, 24 joints
Joints:
- joint j_base_link_haa_RR: origin xyz=-0.215 -0.07 0.0 rpy=0 0 0 -> xyz=-0.215 -0.07world 0.0 rpy=0 0 0
- joint j_kfe_FL: limit (none) -> lower=-2.2 upper=0.0 effort=50 velocity=400; type continuous -> revolute
- joint j_kfe_FR: limit (none) -> lower=0.0 upper=2.2 effort=50 velocity=400; type continuous -> revolute
- joint j_kfe_RL: limit (none) -> lower=-2.2 upper=0.0 effort=50 velocity=400; type continuous -> revolute
- joint j_kfe_RR: limit (none) -> lower=0.0 upper=2.2 effort=50 velocity=400; type continuous -> revolute
