Commit message: Work on estimators.

File: Software/Resource/Robot/Nomad.urdf (robot description, URDF)
Before this commit: robot Nomad, 25 links, 24 joints
Links:
- link b_foot_FL: geometry collision sphere radius=0.025; visual mesh filename=meshes/b_foot_FL.stl scale=0.001 0.001 0.001
- link b_foot_FR: geometry collision sphere radius=0.025; visual mesh filename=meshes/b_foot_FR.stl scale=0.001 0.001 0.001
- link b_foot_RL: geometry collision sphere radius=0.025; visual mesh filename=meshes/b_foot_RL.stl scale=0.001 0.001 0.001
- link b_foot_RR: geometry collision sphere radius=0.025; visual mesh filename=meshes/b_foot_RR.stl scale=0.001 0.001 0.001
- link b_haa_motor_FL: geometry visual mesh filename=meshes/b_haa_motor_FL.stl scale=0.001 0.001 0.001
- link b_haa_motor_FR: geometry visual mesh filename=meshes/b_haa_motor_FR.stl scale=0.001 0.001 0.001
- link b_haa_motor_RL: geometry visual mesh filename=meshes/b_haa_motor_RL.stl scale=0.001 0.001 0.001
- link b_haa_motor_RR: geometry visual mesh filename=meshes/b_haa_motor_RR.stl scale=0.001 0.001 0.001
- link b_hfe_motor_FL: geometry collision cylinder length=0.053 radius=0.05; visual mesh filename=meshes/b_hfe_motor_FL.stl scale=0.001 0.001 0.001
- link b_hfe_motor_FR: geometry collision cylinder length=0.053 radius=0.05; visual mesh filename=meshes/b_hfe_motor_FR.stl scale=0.001 0.001 0.001
- link b_hfe_motor_RL: geometry collision cylinder length=0.053 radius=0.05; visual mesh filename=meshes/b_hfe_motor_RL.stl scale=0.001 0.001 0.001
- link b_hfe_motor_RR: geometry collision cylinder length=0.053 radius=0.05; visual mesh filename=meshes/b_hfe_motor_RR.stl scale=0.001 0.001 0.001
- link b_kfe_motor_FL: geometry collision cylinder length=0.075 radius=0.05; visual mesh filename=meshes/b_kfe_motor_FL.stl scale=0.001 0.001 0.001
- link b_kfe_motor_FR: geometry collision cylinder length=0.075 radius=0.05; visual mesh filename=meshes/b_kfe_motor_FR.stl scale=0.001 0.001 0.001
- link b_kfe_motor_RL: geometry collision cylinder length=0.075 radius=0.05; visual mesh filename=meshes/b_kfe_motor_RL.stl scale=0.001 0.001 0.001
- link b_kfe_motor_RR: geometry collision cylinder length=0.075 radius=0.05; visual mesh filename=meshes/b_kfe_motor_RR.stl scale=0.001 0.001 0.001
- link b_lower_leg_FL: geometry collision cylinder length=0.260 radius=0.01; visual mesh filename=meshes/b_lower_leg_FL.stl scale=0.001 0.001 0.001
- link b_lower_leg_FR: geometry collision cylinder length=0.260 radius=0.01; visual mesh filename=meshes/b_lower_leg_FR.stl scale=0.001 0.001 0.001
- link b_lower_leg_RL: geometry collision cylinder length=0.260 radius=0.01; visual mesh filename=meshes/b_lower_leg_RL.stl scale=0.001 0.001 0.001
- link b_lower_leg_RR: geometry collision cylinder length=0.260 radius=0.01; visual mesh filename=meshes/b_lower_leg_RR.stl scale=0.001 0.001 0.001
- link b_upper_leg_FL: geometry collision box size=.05 .030 .25; visual mesh filename=meshes/b_upper_leg_FL.stl scale=0.001 0.001 0.001
- link b_upper_leg_FR: geometry collision box size=.05 .030 .25; visual mesh filename=meshes/b_upper_leg_FR.stl scale=0.001 0.001 0.001
- link b_upper_leg_RL: geometry collision box size=.05 .030 .25; visual mesh filename=meshes/b_upper_leg_RL.stl scale=0.001 0.001 0.001
- link b_upper_leg_RR: geometry collision box size=.05 .030 .25; visual mesh filename=meshes/b_upper_leg_RR.stl scale=0.001 0.001 0.001
- link base_link: geometry collision box size=0.440 0.260 0.140; visual mesh filename=meshes/base_link.stl scale=0.001 0.001 0.001
Joints:
- joint j_kfe_FL: limit (none) -> lower=-2.2 upper=0.0 effort=50 velocity=400; type continuous -> revolute
- joint j_kfe_FR: limit (none) -> lower=0.0 upper=2.2 effort=50 velocity=400; type continuous -> revolute
- joint j_kfe_RL: limit (none) -> lower=-2.2 upper=0.0 effort=50 velocity=400; type continuous -> revolute
- joint j_kfe_RR: limit (none) -> lower=0.0 upper=2.2 effort=50 velocity=400; type continuous -> revolute

File: Software/Simulation/Gazebo/models/Nomad/Nomad.urdf (robot description, URDF)
Before this commit: robot Nomad, 25 links, 24 joints
Joints:
- joint j_base_link_haa_RR: origin xyz=-0.215 -0.07world 0.0 rpy=0 0 0 -> xyz=-0.215 -0.07 0.0 rpy=0 0 0
