Commit message: Sin Circle Sweep ready to test.

File: Software/Resource/LegTest/Leg Old.urdf (robot description, URDF)
Before this commit: robot Leg, 7 links, 6 joints
Joints:
- joint hfe_to_upper: origin xyz=0.06 0.0 0.000202 rpy=0 0 0 -> xyz=0.06 0.000202 0.0 rpy=0 0 0
- joint j_foot: origin xyz=0.0025 -0.214618 -0.133415 rpy=0 0 0 -> xyz=0.0025 -0.133415 0.214618 rpy=0 0 0
- joint j_kfe: origin xyz=0.0165 0.28 -0.000256 rpy=0 0 0 -> xyz=0.0165 -0.000256 -0.28 rpy=0 0 0
- joint slider: axis 0.0 -0.0 1.0 -> (none); limit lower=0.0 upper=0.0 effort=100 velocity=100 -> (none); type prismatic -> fixed
