Commit message: Adjust Collision Model on URDF

File: Software/Resource/Robot_V2/NOMAD.urdf (robot description, URDF)
Before this commit: robot NOMAD, 25 links, 24 joints
Links:
- removed link b_foot_FL1
- removed link b_foot_FR1
- removed link b_foot_RL1
- removed link b_foot_RL2
- removed link b_haa_motor_FL1
- removed link b_haa_motor_FR1
- removed link b_haa_motor_RL1
- removed link b_haa_motor_RR1
- removed link b_hfe_motor_FL1
- removed link b_hfe_motor_FR1
- removed link b_hfe_motor_RL1
- removed link b_hfe_motor_RR1
- removed link b_kfe_motor_FL1
- removed link b_kfe_motor_FR1
- removed link b_kfe_motor_RL1
- removed link b_kfe_motor_RR1
- removed link b_lower_leg_FL1
- removed link b_lower_leg_FR1
- removed link b_lower_leg_RL1
- removed link b_lower_leg_RR1
- removed link b_upper_leg_FL1
- removed link b_upper_leg_FR1
- removed link b_upper_leg_RL1
- removed link b_upper_leg_RR1
- added link b_foot_FL, mass 0.027943298489902194; collision sphere radius=0.025; visual mesh filename=meshes/b_foot_FL1.dae scale=1.0 1.0 1.0
- added link b_foot_FR, mass 0.027943298489902194; collision sphere radius=0.025; visual mesh filename=meshes/b_foot_FR1.dae scale=1.0 1.0 1.0
- added link b_foot_RL, mass 0.027943298489902197; collision sphere radius=0.025; visual mesh filename=meshes/b_foot_RL2.dae scale=1.0 1.0 1.0
- added link b_foot_RR, mass 0.027943298489902197; collision sphere radius=0.025; visual mesh filename=meshes/b_foot_RL1.dae scale=1.0 1.0 1.0
- added link b_haa_motor_FL, mass 0.7810510004823594; visual mesh filename=meshes/b_haa_motor_FL1.dae scale=1.0 1.0 1.0
- added link b_haa_motor_FR, mass 0.7810510004823594; visual mesh filename=meshes/b_haa_motor_FR1.dae scale=1.0 1.0 1.0
- added link b_haa_motor_RL, mass 0.7810510004823594; visual mesh filename=meshes/b_haa_motor_RL1.dae scale=1.0 1.0 1.0
- added link b_haa_motor_RR, mass 0.7810510004823594; visual mesh filename=meshes/b_haa_motor_RR1.dae scale=1.0 1.0 1.0
- added link b_hfe_motor_FL, mass 0.8403779290245217; visual mesh filename=meshes/b_hfe_motor_FL1.dae scale=1.0 1.0 1.0
- added link b_hfe_motor_FR, mass 0.8403787612467518; visual mesh filename=meshes/b_hfe_motor_FR1.dae scale=1.0 1.0 1.0
- added link b_hfe_motor_RL, mass 0.8403787612467518; visual mesh filename=meshes/b_hfe_motor_RL1.dae scale=1.0 1.0 1.0
- added link b_hfe_motor_RR, mass 0.8403779290245217; visual mesh filename=meshes/b_hfe_motor_RR1.dae scale=1.0 1.0 1.0
- added link b_kfe_motor_FL, mass 0.8552943466477122; visual mesh filename=meshes/b_kfe_motor_FL1.dae scale=1.0 1.0 1.0
- added link b_kfe_motor_FR, mass 0.8552943466477122; visual mesh filename=meshes/b_kfe_motor_FR1.dae scale=1.0 1.0 1.0
- added link b_kfe_motor_RL, mass 0.8552943466477122; visual mesh filename=meshes/b_kfe_motor_RL1.dae scale=1.0 1.0 1.0
- added link b_kfe_motor_RR, mass 0.8552943466477122; visual mesh filename=meshes/b_kfe_motor_RR1.dae scale=1.0 1.0 1.0
- added link b_lower_leg_FL, mass 0.23727593991905244; visual mesh filename=meshes/b_lower_leg_FL1.dae scale=1.0 1.0 1.0
- added link b_lower_leg_FR, mass 0.23727593991905244; visual mesh filename=meshes/b_lower_leg_FR1.dae scale=1.0 1.0 1.0
- added link b_lower_leg_RL, mass 0.23727593991905244; visual mesh filename=meshes/b_lower_leg_RL1.dae scale=1.0 1.0 1.0
- added link b_lower_leg_RR, mass 0.23727593991905244; visual mesh filename=meshes/b_lower_leg_RR1.dae scale=1.0 1.0 1.0
- added link b_upper_leg_FL, mass 0.4893520109323555; visual mesh filename=meshes/b_upper_leg_FL1.dae scale=1.0 1.0 1.0
- added link b_upper_leg_FR, mass 0.4893520109323555; visual mesh filename=meshes/b_upper_leg_FR1.dae scale=1.0 1.0 1.0
- added link b_upper_leg_RL, mass 0.4893520109323555; visual mesh filename=meshes/b_upper_leg_RL1.dae scale=1.0 1.0 1.0
- added link b_upper_leg_RR, mass 0.4893520109323555; visual mesh filename=meshes/b_upper_leg_RR1.dae scale=1.0 1.0 1.0
- link base_link: geometry collision box size=0.402 0.250 0.165; visual mesh filename=meshes/base_link.dae scale=1.0 1.0 1.0
Joints:
- joint j_base_link_haa_FL: child b_haa_motor_FL1 -> b_haa_motor_FL
- joint j_base_link_haa_FR: child b_haa_motor_FR1 -> b_haa_motor_FR
- joint j_base_link_haa_RL: child b_haa_motor_RL1 -> b_haa_motor_RL
- joint j_base_link_haa_RR: child b_haa_motor_RR1 -> b_haa_motor_RR
- joint j_haa_FL: child b_hfe_motor_FL1 -> b_hfe_motor_FL; parent b_haa_motor_FL1 -> b_haa_motor_FL
- joint j_haa_FR: child b_hfe_motor_FR1 -> b_hfe_motor_FR; parent b_haa_motor_FR1 -> b_haa_motor_FR
- joint j_haa_RL: child b_hfe_motor_RL1 -> b_hfe_motor_RL; parent b_haa_motor_RL1 -> b_haa_motor_RL
- joint j_haa_RR: child b_hfe_motor_RR1 -> b_hfe_motor_RR; parent b_haa_motor_RR1 -> b_haa_motor_RR
- joint j_hfe_FL: child b_kfe_motor_FL1 -> b_kfe_motor_FL; parent b_hfe_motor_FL1 -> b_hfe_motor_FL
- joint j_hfe_FR: child b_kfe_motor_FR1 -> b_kfe_motor_FR; parent b_hfe_motor_FR1 -> b_hfe_motor_FR
- joint j_hfe_RL: child b_kfe_motor_RL1 -> b_kfe_motor_RL; parent b_hfe_motor_RL1 -> b_hfe_motor_RL
- joint j_hfe_RR: child b_kfe_motor_RR1 -> b_kfe_motor_RR; parent b_hfe_motor_RR1 -> b_hfe_motor_RR
- joint j_hfe_to_shoulder_FL: child b_upper_leg_FL1 -> b_upper_leg_FL; parent b_kfe_motor_FL1 -> b_kfe_motor_FL
- joint j_hfe_to_shoulder_FR: child b_upper_leg_FR1 -> b_upper_leg_FR; parent b_kfe_motor_FR1 -> b_kfe_motor_FR
- joint j_hfe_to_shoulder_RL: child b_upper_leg_RL1 -> b_upper_leg_RL; parent b_kfe_motor_RL1 -> b_kfe_motor_RL
- joint j_hfe_to_shoulder_RR: child b_upper_leg_RR1 -> b_upper_leg_RR; parent b_kfe_motor_RR1 -> b_kfe_motor_RR
- joint j_kfe_FL: child b_lower_leg_FL1 -> b_lower_leg_FL; parent b_upper_leg_FL1 -> b_upper_leg_FL
- joint j_kfe_FR: child b_lower_leg_FR1 -> b_lower_leg_FR; parent b_upper_leg_FR1 -> b_upper_leg_FR
- joint j_kfe_RL: child b_lower_leg_RL1 -> b_lower_leg_RL; parent b_upper_leg_RL1 -> b_upper_leg_RL
- joint j_kfe_RR: child b_lower_leg_RR1 -> b_lower_leg_RR; parent b_upper_leg_RR1 -> b_upper_leg_RR
- joint j_knee_to_foot_FL: child b_foot_FL1 -> b_foot_FL; parent b_lower_leg_FL1 -> b_lower_leg_FL
- joint j_knee_to_foot_FR: child b_foot_FR1 -> b_foot_FR; parent b_lower_leg_FR1 -> b_lower_leg_FR
- joint j_knee_to_foot_RL: child b_foot_RL2 -> b_foot_RL; parent b_lower_leg_RL1 -> b_lower_leg_RL
- joint j_knee_to_foot_RR: child b_foot_RL1 -> b_foot_RR; parent b_lower_leg_RR1 -> b_lower_leg_RR

Commit message: Full Test of new URDF + Stand.

File: Software/Resource/Robot_V2/NOMAD.urdf (robot description, URDF)
Before this commit: robot NOMAD, 25 links, 24 joints
Links:
- link b_foot_RL: mass 0.027943298489902197 -> 0.027943298489902194; geometry collision sphere radius=0.025; visual mesh filename=meshes/b_foot_RL.dae scale=1.0 1.0 1.0
Joints:
- joint j_kfe_FR: axis 0.0 -1.0 -0.0 -> 0.0 1.0 -0.0
- joint j_kfe_RR: axis -0.0 -1.0 0.0 -> -0.0 1.0 0.0
- joint j_knee_to_foot_RL: origin xyz=0.211714 -0.3425 -0.138133 rpy=0 0 0 -> xyz=0.211714 -0.0 -0.138133 rpy=0 0 0

Commit message: Add Watchdog Timers back.  Adjust URDF

File: Software/Resource/Robot_V2/NOMAD.urdf (robot description, URDF)
Before this commit: robot NOMAD, 25 links, 24 joints
Links:
- link b_lower_leg_FL: geometry collision mesh filename=meshes/b_lower_leg_FL1.dae scale=1.0 1.0 1.0; visual mesh filename=meshes/b_lower_leg_FL1.dae scale=1.0 1.0 1.0
- link b_lower_leg_FR: geometry collision mesh filename=meshes/b_lower_leg_FR1.dae scale=1.0 1.0 1.0; visual mesh filename=meshes/b_lower_leg_FR1.dae scale=1.0 1.0 1.0
- link b_lower_leg_RL: geometry collision mesh filename=meshes/b_lower_leg_RL1.dae scale=1.0 1.0 1.0; visual mesh filename=meshes/b_lower_leg_RL1.dae scale=1.0 1.0 1.0
- link b_lower_leg_RR: geometry collision mesh filename=meshes/b_lower_leg_RR1.dae scale=1.0 1.0 1.0; visual mesh filename=meshes/b_lower_leg_RR1.dae scale=1.0 1.0 1.0
